File: CAD/DropGen_PCB/DropGenPCB.kicad_pcb (KiCad board)
At the start: 2 copper layers, 92.5 x 62.5 mm, 25 parts, among them J1 JST_3_pin, J2 JST_4_pin, J3 Barrel_Jack_Switch, J4 Camera Terminal Block, J5 Piezo, U1 SEEED XIAO ESP32S3, U2 TMC2209_SILENTSTEPSTICK, U3 L293D, U4 TPS5430DDAR

Commit message: updated BOM and CPL
Parts:
- L1: value 22uH -> 22uH

Commit message: now saves values locally between restarts.
Connections:
- net IN3 renamed SERVO
- U3 pad 3: Piezo 2 -> unconnected-(U3-OUT3-Pad3)
- U3 pad 6: Piezo 1 -> unconnected-(U3-OUT4-Pad6)
- U3 pad 7: IN4 -> unconnected-(U3-IN4-Pad7)
Changed lines of the file:
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@@
 	(net 13 "STEP")
 	(net 14 "DIR")
-	(net 15 "IN3")
+	(net 15 "SERVO")
 	(net 16 "IN4")
 	(net 17 "unconnected-(U1-D0-Pad1)")
@@
 	(net 34 "Net-(U2-M2A)")
 	(net 35 "Net-(D2-A)")
+	(net 36 "unconnected-(U3-IN4-Pad7)")
+	(net 37 "unconnected-(U3-OUT3-Pad3)")
+	(net 38 "unconnected-(U3-OUT4-Pad6)")
 	(footprint "DropGeneratorPCB:ESP32S3"
 		(layer "F.Cu")
@@
 			(layers "*.Cu" "*.Mask")
 			(remove_unused_layers no)
-			(net 15 "IN3")
+			(net 15 "SERVO")
 			(pinfunction "D3")
 			(pintype "bidirectional")
@@
 			(layers "*.Cu" "*.Mask")
 			(remove_unused_layers no)
-			(net 15 "IN3")
+			(net 15 "SERVO")
 			(pinfunction "IN3")
 			(pintype "input")
@@
 			(layers "*.Cu" "*.Mask")
 			(remove_unused_layers no)
-			(net 11 "Piezo 2")
+			(net 37 "unconnected-(U3-OUT3-Pad3)")
 			(pinfunction "OUT3")
-			(pintype "output")
+			(pintype "output+no_connect")
 		)
 		(pad "4" thru_hole oval
@@
 			(layers "*.Cu" "*.Mask")
 			(remove_unused_layers no)
-			(net 10 "Piezo 1")
+			(net 38 "unconnected-(U3-OUT4-Pad6)")
 			(pinfunction "OUT4")
-			(pintype "output")
+			(pintype "output+no_connect")
 		)
 		(pad "7" thru_hole oval
@@
 			(layers "*.Cu" "*.Mask")
 			(remove_unused_layers no)
-			(net 16 "IN4")
+			(net 36 "unconnected-(U3-IN4-Pad7)")
 			(pinfunction "IN4")
-			(pintype "input")
+			(pintype "input+no_connect")
 		)
 		(pad "8" thru_hole rect
